Commit message: ball_detection works

File: src/final_description/urdf/final_1.urdf (robot description, URDF)
Before this commit: robot bot1, 14 links, 13 joints
Links:
- added link LC, mass 0.075; collision mesh filename=package://final_description/meshes/LC.STL; visual mesh filename=package://final_description/meshes/LC.STL
- added link RC, mass 0.075; collision mesh filename=package://final_description/meshes/RC.STL; visual mesh filename=package://final_description/meshes/RC.STL
- link base_link: geometry collision mesh filename=package://final_description/meshes/base_link.STL; visual mesh filename=package://final_description/meshes/base_link.STL
Joints:
- added joint LCJ: type fixed, parent base_link, child LC, origin xyz=0.03 0.23 0.125 rpy=-1.5707963267949 0 -1.5707963267949, axis 0 0 0
- added joint RCJ: type fixed, parent base_link, child RC, origin xyz=0.03 -0.23 0.125 rpy=1.5707963267949 0 1.5707963267949, axis 0 0 0
- joint FCJ: origin xyz=0.01 0.275 0 rpy=-1.57 0 0 -> xyz=0.01 0.275 0 rpy=0 0 0
- joint LFJ: limit lower=-0.34 upper=1.36 effort=100 velocity=0.15 -> lower=-0.34 upper=1.36 effort=100 velocity=0.125; mimic joint=RFJ multiplier=-1 offset=0 -> (none)
- joint RFJ: limit lower=-1.5 upper=0.2 effort=100 velocity=0.15 -> lower=-1.5 upper=0.2 effort=100 velocity=0.125
